File: hardware/level-shifter/level-shifter.kicad_sch (KiCad schematic)
At the start: 47 parts, among them IC1 NXB0104PW-Q100J, IC10 NXB0104PW-Q100J, IC2 NXB0104PW-Q100J, IC3 NXB0104PW-Q100J, IC4 NXB0104PW-Q100J, IC5 NXB0104PW-Q100J, IC6 NXB0104PW-Q100J, IC7 NXB0104PW-Q100J, IC8 NXB0104PW-Q100J, IC9 NXB0104PW-Q100J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

Commit message: changed PCB to include FlipFlop
Parts:
- removed C22: 100nF, Capacitor_SMD:C_0805_2012Metric, symbol Device:C
- added C23: 100nF, Capacitor_SMD:C_0805_2012Metric, symbol Device:C
- added U2: CD74AC109M96, D16, symbol CD74AC109M96:CD74AC109M96
Connections:
- net +3V3UL: now also C21.2, U1.2 (VDD), C23.1, U2.1 (*1CLR), U2.16 (VCC), U2.2 (1J), U2.5 (*1PRE)
- net +5V: no longer C21.2, U1.2 (VDD), U1.7 (OE)
- net GND: now also U1.4 (S1), U1.6 (S0), C23.2, U2.3 (*1K), U2.8 (GND)
- net PLLCLK: now also U2.4 (1CLK); no longer J1.13 (Pin_13)
- new net DOUBLE_CLK: J1.13 (Pin_13), U2.6 (1Q)
- no-connect marks 69 -> 76
Other:
- note added: "<--- Clock Multiplier Does x4 to get clock from 4MHz to 16MHz"
- note added: "<--- JK Flip Flop Does /2 to get clock from 16MHz to 8MHz"
- moved on the sheet: C21, U1

Commit message: added tester board files
Parts:
- U2: footprint D16 -> CD74AC109M96:CD74AC109M96
Changed lines of the file:
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@@
 			)
 		)
-		(property "Footprint" "D16"
+		(property "Footprint" "CD74AC109M96:CD74AC109M96"
 			(at 264.16 311.15 0)
 			(effects
