File: TesterBoard/Tester/untitled.kicad_sch (KiCad schematic)
At the start: 4 parts, among them U3 74LS04, U4 sn74ls32n, U5 CY62256-70PC, U6 28C256

Commit message: pcb stuff
Connections:
- no-connect marks 2 -> 1

Commit message: schematic done
Parts:
- removed U3: 74LS04, symbol 74xx:74LS04
- removed U6: 28C256, symbol Memory_EEPROM:28C256
- added C10, C11, C12, C13, C3, C6, C7, C8, C9: 100nF, Capacitor_THT:CP_Radial_D4.0mm_P2.00mm, symbol Device:C
- added DS1: NHD-12864WG-BTMI-V#N, Z80_Tester_Footprints:NHD12864WGBTMIVN, symbol displays:NHD-12864WG-BTMI-V#N
- added R10, R11, R12, R13, R14, R15, R8, R9: 10K, ECE445L:R_Axial_DIN0204_L3.6mm_D1.6mm_P7.62mm_Horizontal, symbol Device:R
- added R3: 1K, ECE445L:R_Axial_DIN0204_L3.6mm_D1.6mm_P7.62mm_Horizontal, symbol Device:R
- added RV1, RV2: R_Potentiometer, Potentiometer_THT:Potentiometer_Alps_RK163_Single_Horizontal, symbol Device:R_Potentiometer
- added S1, S3, S4, S5, S6, S7, S8, S9: B3F-4050, Button_Switch_THT:SW_PUSH_6mm, symbol Switch:SW_Push
- added U10: 74HC244, Package_DIP:DIP-20_W7.62mm, symbol 74xx:74HC244
- added U3: 74LS14, Package_DIP:DIP-14_W7.62mm_Socket, symbol 74xx:74LS14
- added U6: LCD-16X2, Z80_Tester_Footprints:MODULE_LCD-16X2, symbol displays:LCD-16X2
- added U7: SST39SF010, Socket:DIP_Socket-32_W11.9_W12.7_W15.24_W17.78_W18.5_3M_232-1285-00-0602J, symbol Memory_Flash:SST39SF010
- added U8: 74HC138, Package_DIP:DIP-16_W7.62mm_Socket, symbol 74xx:74HC138
- added U9: 74HC00, Package_DIP:DIP-14_W7.62mm_Socket, symbol 74xx:74HC00
- U4: footprint (none) -> Package_DIP:DIP-14_W7.62mm_Socket
Connections:
- net +5V: now also U5.28 (VCC), C10.2, C11.2, C12.1, C13.2, C3.1, C6.2, C7.1, C8.2, C9.2, DS1.1 (VDD), DS1.14 (~{RST}), R10.1, R11.1, R12.1, R13.1, R14.1, R15.1, R3.1, R8.1, R9.1, RV1.1, U10.20 (VCC), U3.11, U3.13, U3.14 (VCC), U6.15 (A), U6.2 (VDD), U7.31 (PGM), U7.32 (VCC), U8.16 (VCC), U8.6 (E2), U9.14 (VCC)
- net Address0: now also U7.12 (A0), U8.1 (A0)
- net Address1: now also U7.11 (A1), U8.2 (A1)
- net Address10: now also U7.23 (A10)
- net Address11: now also U7.25 (A11)
- net Address12: now also U7.4 (A12)
- net Address13: now also U7.28 (A13)
- net Address14: now also U7.29 (A14)
- net Address15: now also U3.1, U7.24 (OE), U7.3 (A15)
- net Address2: now also U7.10 (A2), U8.3 (A2)
- net Address3: now also DS1.16 (D/~{I}), U6.4 (RS), U7.9 (A3)
- net Address4: now also DS1.13 (CS2), U3.5, U7.8 (A4)
- net Address5: now also U7.7 (A5)
- net Address6: now also U7.6 (A6)
- net Address7: now also U7.5 (A7)
- net Address8: now also U7.27 (A8)
- net Address9: now also U7.26 (A9)
- net Data0: now also DS1.4 (DB0), U10.18 (1Y0), U6.7 (DB0), U7.13 (D0)
- net Data1: now also DS1.5 (DB1), U10.16 (1Y1), U6.8 (DB1), U7.14 (D1)
- net Data2: now also DS1.6 (DB2), U10.14 (1Y2), U6.9 (DB2), U7.15 (D2)
- net Data3: now also DS1.7 (DB3), U10.12 (1Y3), U6.10 (DB3), U7.17 (D3)
- net Data4: now also DS1.8 (DB4), U10.3 (2Y0), U6.11 (DB4), U7.18 (D4)
- net Data5: now also DS1.9 (DB5), U10.5 (2Y1), U6.12 (DB5), U7.19 (D5)
- net Data6: now also DS1.10 (DB6), U10.7 (2Y2), U6.13 (DB6), U7.20 (D6)
- net Data7: now also DS1.11 (DB7), U10.9 (2Y3), U6.14 (DB7), U7.21 (D7)
- net GND: now also U5.14 (GND), C10.1, C11.1, C12.2, C13.1, C3.2, C6.1, C7.2, C8.1, C9.1, DS1.15 (R/~{W}), DS1.2 (VSS), DS1.20 (K), RV1.3, RV2.3, S1.2, S3.2, S4.2, S5.2, S6.2, S7.2, S8.2, S9.2, U10.10 (GND), U10.11 (2A3), U10.13 (2A2), U10.15 (2A1), U10.17 (2A0), U10.2 (1A0), U10.4 (1A1), U10.6 (1A2), U10.8 (1A3), U3.7 (GND), U6.1 (VSS), U6.16 (K), U6.5 (R/W), U7.16 (GND), U7.2 (A16), U8.5 (~{E1}), U8.8 (GND), U9.12, U9.13, U9.7 (GND)
- net /RD: now also U9.10
- net /WR: now also U3.3, U9.2, U9.5
- net at U5.20 (~{CS}): now also U3.2
- net at U4.3, U5.22 (~{OE}): now also U7.22 (CE)
- new net: R8.2, S1.1
- new net: DS1.3 (V0), RV2.2
- new net: R15.2, S9.1
- new net: DS1.19 (A), R3.2
- new net: R14.2, S8.1
- new net: R10.2, S4.1
- new net: R12.2, S6.1
- new net: R9.2, S3.1
- new net: RV1.2, U6.3 (VO)
- new net: R11.2, S5.1
- new net: R13.2, S7.1
- new net 12864_Enable: DS1.17 (E), U9.6
- new net 12864_VEE: DS1.18 (VEE), RV2.1
- new net 1602_Enable: U6.6 (E), U9.3
- new net Buttons_Enable: U3.9, U9.8
- new net \WR_inv: U3.4
- new net /12864_Select: U8.14 (~{Y1}), U9.4
- new net /1602_Select: U8.15 (~{Y0}), U9.1
- new net /Address4: DS1.12 (CS1), U3.6
- new net /Buttons_Enable: U10.1 (1OE), U10.19 (2OE), U3.8
- new net /Buttons_Select: U8.13 (~{Y2}), U9.9
- new net /IOREQ: U8.4 (~{E0})
- no-connect marks 1 -> 16
Other:
- note added: "12864 LCD"
- note added: "1602 LCD"
- note added: "IO 3-8 Decoder"
- note added: "IO Enable Logic"
- note added: "Input Buttons"
- note added: "Schmitt Trigger Inverter"
- moved on the sheet: U4C
